Commit message: Add joystick teleop for MPSF and direct modes on sim and hardware.
Introduce teleop:=mpsf|direct|none with shared joy helpers, stick-enable
gating, gripper toggle, and arm differential IK. Direct teleop publishes
synthetic MpcPlans to the low-level tracker without running MPC; MPSF/MPC
teleop drives desired velocity with soft obstacle costs, base velocity
guarding, and smoother plan tracking. Add hardware_teleop.launch plus
configs for obstacle teleop, tray balancing (empty/clutter), tray hold,
and matching docs/tests.

File: mm_assets/thing/xacro/collision.urdf.xacro (robot description, xacro)
@@ -43,7 +43,7 @@
   </xacro:macro>
   <!-- Collision sphere for the base -->
-  <xacro:collision_link_sphere name="base_collision_link" radius="0.55"/>
+  <xacro:collision_link_sphere name="base_collision_link" radius="0.49"/>
   <joint name="base_collision_joint" type="fixed">
-    <origin rpy="0 0 0" xyz="0 0 -0.08"/>
+    <origin rpy="0 0 0" xyz="0 0 0"/>
     <parent link="base_link"/>
     <child link="base_collision_link"/>

Commit message: Harden teleop: world-frame sticks, idle vel gate, and gripper/tray collisions.
Map chassis-frame joystick twists into world frame, zero near-idle measured
base/arm velocity before MPC, and split thing vs thing_tray collision models
(gripper spheres + optional tray). Rename cluttered scene configs and fix
d-pad EE yaw button indices.

File: mm_assets/thing/xacro/collision.urdf.xacro (robot description, xacro)
@@ -23,5 +23,5 @@
     </link>
   </xacro:macro>
-    <xacro:macro name="collision_link_cylinder" params="name radius">
+    <xacro:macro name="collision_link_cylinder" params="name radius length">
     <link name="${name}">
       <xacro:if value="$(arg use_collision)">
@@ -29,5 +29,5 @@
           <origin rpy="0 0 0" xyz="0 0 0" />
           <geometry>
-            <cylinder  radius="${radius}" length="1"/>
+            <cylinder radius="${radius}" length="${length}"/>
           </geometry>
         </collision>
@@ -36,5 +36,5 @@
         <origin rpy="0 0 0" xyz="0 0 0" />
         <geometry>
-          <cylinder  radius="${radius}" length="1"/>
+          <cylinder radius="${radius}" length="${length}"/>
         </geometry>
         <material name="${material}"/>
@@ -61,5 +61,5 @@
     <child link="base_collision_link_back"/>
   </joint> -->
-  <xacro:collision_link_cylinder name="rack_collision_link" radius="0.325"/>
+  <xacro:collision_link_cylinder name="rack_collision_link" radius="0.325" length="1"/>
   <joint name="rack_collision_joint" type="fixed">
     <origin rpy="0 0 0" xyz="-0.45 -0. 0.75"/>
@@ -136,10 +136,18 @@
     <child link="ur10_arm_wrist3_collision_link"/>
   </joint>
-  <!-- Gripped Object -->
-  <xacro:collision_link_sphere name="gripped_object_collision_link" radius="0.15"/>
-  <joint name="gripped_object_collision_joint" type="fixed">
-    <origin rpy="0 0 0" xyz="0 0 0.0"/>
-    <parent link="gripped_object"/>
-    <child link="gripped_object_collision_link"/>
+  <!-- Robotiq gripper: 3" shaft + 3.5"-diameter palm as spheres (fingers unmodeled).
+       Shaft sphere circumscribes the old cylinder (r=0.045, L=0.076) at z=0.038.
+       Palm center at z=0.121. Spheres keep MPC on sphere–sphere / sphere–cylinder. -->
+  <xacro:collision_link_sphere name="gripper_shaft_collision_link" radius="0.059"/>
+  <joint name="gripper_shaft_collision_joint" type="fixed">
+    <origin rpy="0 0 0" xyz="0 0 0.038"/>
+    <parent link="gripper"/>
+    <child link="gripper_shaft_collision_link"/>
+  </joint>
+  <xacro:collision_link_sphere name="gripper_palm_collision_link" radius="0.0445"/>
+  <joint name="gripper_palm_collision_joint" type="fixed">
+    <origin rpy="0 0 0" xyz="0 0 0.121"/>
+    <parent link="gripper"/>
+    <child link="gripper_palm_collision_link"/>
   </joint>
 </robot>

File: mm_assets/thing/xacro/end_effector_empty.urdf.xacro (robot description, xacro)
@@ -1,43 +1,26 @@
 <?xml version="1.0" encoding="utf-8"?>
-<robot name="end_effector_fingers" xmlns:xacro="http://wiki.ros.org/xacro">
-<!--  <joint name="tool0_tcp_fixed_joint" type="fixed">-->
-<!--    <origin rpy="0.0 0.0 3.14159" xyz="0.0 0.0 0.290"/>-->
-<!--    <parent link="ur10_arm_tool0"/>-->
-<!--    <child link="thing_tool"/>-->
-<!--  </joint>-->
-  <!-- s = 0.3 -->
-  <!-- h = 0.08660254037844387 -->
-  <!-- r = 0.17320508075688773 -->
-  <!-- s = 0.2 -->
-  <!-- h = 0.0577 -->
-  <!-- r = 0.1155 -->
-   <joint name="gripped_object_joint" type="fixed">
-     <xacro:transformed_origin name="gripped_object_transform" />
-     <parent link="gripper"/>
-     <child link="gripped_object"/>
-   </joint>
-  <!-- Custom tool for tray balancing -->
-  <!-- When oriented forward, the frame has: z forward, x down, y left -->
-  <!-- When oriented up (i.e. for balancing): z up, x forward, y left -->
+<robot name="end_effector_empty" xmlns:xacro="http://wiki.ros.org/xacro">
+  <!-- TCP / fingertips frame (~0.29 m from gripper). Visual marker only; MPC
+       collision for the hand lives on gripper_* links in collision.urdf.xacro. -->
+  <joint name="gripped_object_joint" type="fixed">
+    <xacro:transformed_origin name="gripped_object_transform" />
+    <parent link="gripper"/>
+    <child link="gripped_object"/>
+  </joint>
+  <!-- When oriented forward: z forward, x down, y left.
+       When oriented up (balancing): z up, x forward, y left. -->
   <link name="gripped_object">
     <visual>
-      <origin rpy="0 0 0" xyz="0.0 0 0"/>
+      <origin rpy="0 0 0" xyz="0 0 0"/>
       <geometry>
         <sphere radius="0.02"/>
       </geometry>
-      <material name="green">
+      <material name="tcp_marker">
         <color rgba="1 0 0 1"/>
       </material>
     </visual>
-    <collision>
-      <origin rpy="0 0 0" xyz="0.0 0 0"/>
-      <geometry>
-        <sphere radius="0.02"/>
-      </geometry>
-    </collision>
     <inertial>
       <origin rpy="0 0 0" xyz="0 0 0"/>
       <mass value="0.1"/>
-      <!-- not accurate, but pybullet recomputes this by default -->
       <inertia ixx="1" ixy="0" ixz="0" iyy="1" iyz="0" izz="1"/>
     </inertial>

File: mm_assets/thing/xacro/end_effector_fingers.urdf.xacro (robot description, xacro)
@@ -1,23 +1,11 @@
 <?xml version="1.0" encoding="utf-8"?>
 <robot name="end_effector_fingers" xmlns:xacro="http://wiki.ros.org/xacro">
-<!--  <joint name="tool0_tcp_fixed_joint" type="fixed">-->
-<!--    <origin rpy="0.0 0.0 3.14159" xyz="0.0 0.0 0.290"/>-->
-<!--    <parent link="ur10_arm_tool0"/>-->
-<!--    <child link="thing_tool"/>-->
-<!--  </joint>-->
-  <!-- s = 0.3 -->
-  <!-- h = 0.08660254037844387 -->
-  <!-- r = 0.17320508075688773 -->
-  <!-- s = 0.2 -->
-  <!-- h = 0.0577 -->
-  <!-- r = 0.1155 -->
-   <joint name="gripped_object_joint" type="fixed">
-     <xacro:transformed_origin name="gripped_object_transform" />
-     <parent link="gripper"/>
-     <child link="gripped_object"/>
-   </joint>
-  <!-- Custom tool for tray balancing -->
-  <!-- When oriented forward, the frame has: z forward, x down, y left -->
-  <!-- When oriented up (i.e. for balancing): z up, x forward, y left -->
+  <!-- Legacy fingertip markers (visual only). Prefer end_effector_empty for
+       gripper-only MPC; collision is on gripper_* links. -->
+  <joint name="gripped_object_joint" type="fixed">
+    <xacro:transformed_origin name="gripped_object_transform" />
+    <parent link="gripper"/>
+    <child link="gripped_object"/>
+  </joint>
   <link name="gripped_object">
     <visual>
@@ -44,26 +32,7 @@
       <material name="red"/>
     </visual>
-    <collision>
-      <origin rpy="0 0 0" xyz="0.1155 0 0"/>
-      <geometry>
-        <sphere radius="0.02"/>
-      </geometry>
-    </collision>
-    <collision>
-      <origin rpy="0 0 0" xyz="-0.0577 0.1 0"/>
-      <geometry>
-        <sphere radius="0.02"/>
-      </geometry>
-    </collision>
-    <collision>
-      <origin rpy="0 0 0" xyz="-0.0577 -0.1 0"/>
-      <geometry>
-        <sphere radius="0.02"/>
-      </geometry>
-    </collision>
     <inertial>
       <origin rpy="0 0 0" xyz="0 0 0"/>
       <mass value="0.1"/>
-      <!-- not accurate, but pybullet recomputes this by default -->
       <inertia ixx="1" ixy="0" ixz="0" iyy="1" iyz="0" izz="1"/>
     </inertial>

File: mm_assets/thing/xacro/end_effector_tray_gripped.urdf.xacro (robot description, xacro)
@@ -1,4 +1,12 @@
 <?xml version="1.0" encoding="utf-8"?>
 <robot name="end_effector_tray_gripped" xmlns:xacro="http://wiki.ros.org/xacro">
+  <!-- Square tray 11.5" side, 3" thick. Visual is a flat cylinder; MPC collision
+       is a conservative circumscribed sphere (avoids cylinder–cylinder SD).
+       TCP at gripped_object (~fingertips).
+       use_collision comes from robot urdf args (declared in collision.urdf.xacro). -->
+  <xacro:property name="tray_disk_radius" value="0.2065"/>
+  <xacro:property name="tray_height" value="0.076"/>
+  <!-- sqrt(R^2 + (H/2)^2) for R=0.2065, H=0.076 -->
+  <xacro:property name="tray_collision_radius" value="0.210"/>
   <joint name="gripped_object_joint" type="fixed">
     <xacro:transformed_origin name="gripped_object_transform" />
@@ -8,7 +16,7 @@
   <link name="gripped_object">
     <visual>
-      <origin rpy="0 0 0" xyz="0 0 -0.01"/>
+      <origin rpy="0 0 0" xyz="0 0 0"/>
       <geometry>
-        <cylinder length="0.02" radius="0.16"/>
+        <cylinder length="${tray_height}" radius="${tray_disk_radius}"/>
       </geometry>
       <material name="tray_black">
@@ -16,10 +24,4 @@
       </material>
     </visual>
-    <collision>
-      <origin rpy="0 0 0" xyz="0 0 -0.01"/>
-      <geometry>
-        <cylinder length="0.02" radius="0.16"/>
-      </geometry>
-    </collision>
     <inertial>
       <origin rpy="0 0 0" xyz="0 0 0"/>
@@ -28,3 +30,26 @@
     </inertial>
   </link>
+  <!-- Separate named link for MPC collision_link_names.tool -->
+  <link name="tray_collision_link">
+    <xacro:if value="$(arg use_collision)">
+      <collision>
+        <origin rpy="0 0 0" xyz="0 0 0"/>
+        <geometry>
+          <sphere radius="${tray_collision_radius}"/>
+        </geometry>
+      </collision>
+    </xacro:if>
+    <visual>
+      <origin rpy="0 0 0" xyz="0 0 0"/>
+      <geometry>
+        <sphere radius="${tray_collision_radius}"/>
+      </geometry>
+      <material name="seethrough"/>
+    </visual>
+  </link>
+  <joint name="tray_collision_joint" type="fixed">
+    <origin rpy="0 0 0" xyz="0 0 0"/>
+    <parent link="gripped_object"/>
+    <child link="tray_collision_link"/>
+  </joint>
 </robot>

Commit message: Unify teleop by task and stabilize pick-place RL and gripper.
Replace per-mode experiment YAMLs with teleop_pick_place and teleop_tray so mpsf/direct/rl share one config. Tighten collision geometry (Ridgeback footprint, rack poles, gripped object), add an orientation curriculum and min-α floor so SAC does not collapse, and seed Robotiq commands from status so Triangle does not force a mode-change dance.

File: mm_assets/thing/xacro/collision.urdf.xacro (robot description, xacro)
@@ -42,38 +42,41 @@
     </link>
   </xacro:macro>
-  <!-- Collision sphere for the base -->
-  <xacro:collision_link_sphere name="base_collision_link" radius="0.49"/>
+  <!-- Unused single circumscribed base sphere (prefer front+back below). -->
+  <!-- <xacro:collision_link_sphere name="base_collision_link" radius="0.49"/>
   <joint name="base_collision_joint" type="fixed">
     <origin rpy="0 0 0" xyz="0 0 0"/>
     <parent link="base_link"/>
     <child link="base_collision_link"/>
-  </joint>
-  <!-- <xacro:collision_link_sphere name="base_collision_link_front" radius="0.3"/>
+  </joint> -->
+  <!-- Two spheres for rounded-rect Ridgeback footprint (less conservative than r=0.49). -->
+  <xacro:collision_link_sphere name="base_collision_link_front" radius="0.39"/>
   <joint name="base_collision_joint_front" type="fixed">
-    <origin rpy="0 0 0" xyz="0.35 0 -0.08"/>
+    <origin rpy="0 0 0" xyz="0.1 0 0.1"/>
     <parent link="base_link"/>
     <child link="base_collision_link_front"/>
   </joint>
-  <xacro:collision_link_sphere name="base_collision_link_back" radius="0.3"/>
+  <xacro:collision_link_sphere name="base_collision_link_back" radius="0.39"/>
   <joint name="base_collision_joint_back" type="fixed">
-    <origin rpy="0 0 0" xyz="-0.25 0 -0.08"/>
+    <origin rpy="0 0 0" xyz="-0.05 0 0.1"/>
     <parent link="base_link"/>
     <child link="base_collision_link_back"/>
-  </joint> -->
-  <xacro:collision_link_cylinder name="rack_collision_link" radius="0.325" length="1"/>
+  </joint>
+  <!-- Unused cylinder (not listed under collision_link_names.rack). -->
+  <!-- <xacro:collision_link_cylinder name="rack_collision_link" radius="0.325" length="1"/>
   <joint name="rack_collision_joint" type="fixed">
     <origin rpy="0 0 0" xyz="-0.45 -0. 0.75"/>
     <parent link="base_link"/>
     <child link="rack_collision_link"/>
-  </joint>
-  <xacro:collision_link_sphere name="rack_collision_link_sphere_1" radius="0.5"/>
+  </joint> -->
+  <!-- Rear rack poles: small spheres ~5 cm past back, ~10 cm in from sides, z=0.25. -->
+  <xacro:collision_link_sphere name="rack_collision_link_sphere_1" radius="0.05"/>
   <joint name="rack_collision_joint_1" type="fixed">
-    <origin rpy="0 0 0" xyz="-0.45 -0.15 0.75"/>
+    <origin rpy="0 0 0" xyz="-0.45 -0.25 0.25"/>
     <parent link="base_link"/>
     <child link="rack_collision_link_sphere_1"/>
   </joint>
-  <xacro:collision_link_sphere name="rack_collision_link_sphere_2" radius="0.5"/>
+  <xacro:collision_link_sphere name="rack_collision_link_sphere_2" radius="0.05"/>
   <joint name="rack_collision_joint_2" type="fixed">
-    <origin rpy="0 0 0" xyz="-0.45 0.15 0.75"/>
+    <origin rpy="0 0 0" xyz="-0.45 0.25 0.25"/>
     <parent link="base_link"/>
     <child link="rack_collision_link_sphere_2"/>
@@ -130,5 +133,5 @@
     <child link="ur10_arm_wrist1_collision_link"/>
   </joint>
-  <xacro:collision_link_sphere name="ur10_arm_wrist3_collision_link" radius="0.2"/>
+  <xacro:collision_link_sphere name="ur10_arm_wrist3_collision_link" radius="0.15"/>
   <joint name="ur10_arm_wrist3_collision_joint" type="fixed">
     <origin rpy="0 0 0" xyz="0 0 0"/>
@@ -151,3 +154,10 @@
     <child link="gripper_palm_collision_link"/>
   </joint>
+  <!-- Gripped object / fingertips ahead of palm along gripper +Z (moves with EE). -->
+  <xacro:collision_link_sphere name="gripped_object_collision_link" radius="0.05"/>
+  <joint name="gripped_object_collision_joint" type="fixed">
+    <origin rpy="0 0 0" xyz="0 0 0.22"/>
+    <parent link="gripper"/>
+    <child link="gripped_object_collision_link"/>
+  </joint>
 </robot>
