Commit message: Final YAMLs, adding cable guard, adding CSV exports and plotting

File: mm_assets/thing/xacro/end_effector_tray_gripped.urdf.xacro (robot description, xacro)
@@ -8,5 +8,5 @@
   <xacro:property name="tray_height" value="0.076"/>
   <!-- sqrt(R^2 + (H/2)^2) for R=0.2065, H=0.076 -->
-  <xacro:property name="tray_collision_radius" value="0.210"/>
+  <xacro:property name="tray_collision_radius" value="0.18"/>
   <joint name="gripped_object_joint" type="fixed">
     <xacro:transformed_origin name="gripped_object_transform" />
